File: PCB/GlowBit-Rainbow.kicad_pcb (KiCad board)
At the start: 2 copper layers, 76.2 x 42.7 mm, 24 parts, among them J1 3V, J2 data, J3 G, J4 Conn_01x04_Male

Commit message: Version 1.2
Correct the rear silk pin labels (DI and DO were swapped in v1.1)
Other:
- board text added: "v1.2"
- board text removed: "v1.1"
