File: PCB/GlowBit-Rainbow.sch (KiCad schematic (older format))
At the start: 24 parts, among them J1 3V, J2 data, J3 G, J4 Conn_01x04_Male

Commit message: Version 1.2
Correct the rear silk pin labels (DI and DO were swapped in v1.1)
Parts:
- J4: value Conn_01x04_Male -> (none)
Changed lines of the file:
@@
 Sheet 1 1
 Title "GlowBit Rainbow"
-Date "2020-12-15"
-Rev "1.1"
+Date "2021-03-22"
+Rev "1.2"
 Comp "Core Electronics"
 Comment1 "Designed at Core Electronics by Michael Ruppe"
 Comment2 "License: CCASAv4.0 https://creativecommons.org/licenses/by-sa/4.0/"
 Comment3 "Released under the Creative Commons Attribution Share-Alike 4.0 License"
-Comment4 "A delightful rainbow of colour"
+Comment4 "\"GlowBit\" is a trademark of Core Electronics Pty Ltd"
 $EndDescr
 $Comp
@@
 P 850 4650
 F 0 "J4" H 958 4931 50  0000 C CNN
-F 1 "Conn_01x04_Male" H 958 4840 50  0000 C CNN
+F 1 " " H 958 4840 50  0000 C CNN
 F 2 "Connector_PinSocket_2.54mm:PinSocket_1x04_P2.54mm_Vertical" H 850 4650 50  0001 C CNN
 F 3 "~" H 850 4650 50  0001 C CNN
